File: FoC Motor Controller.kicad_sch (KiCad schematic)
At the start: 0 parts

Commit message: Reorganize project into Altium-style folder structure; add README
- Move hierarchical sheets to Schematics/, lib/ -> Libraries/,
  Manufacturing/ -> Project Outputs/ (BOM, Assembly, Netlist,
  Fabrication, PDF), LTspice benches -> Simulation/
- Update Sheetfile, ${KIPRJMOD} library/3D-model, and output paths
- Drop unused sheets, datasheets, templates and KiCad local history
  from the tracked tree (kept locally, now in .gitignore)
- README.md is the design build log

Co-Authored-By: Claude Sonnet 5 <noreply@anthropic.com>
Other:
- removed sheet Block Diagram
- removed sheet Power - Sequencing
- removed sheet Revision History
- sheet Project Architecture: file Project Architecture.kicad_sch -> Schematics/Project Architecture.kicad_sch
- note added: "Interface - CAN FD"
- note added: "Interface - Interconnects"
- note added: "MCU - IOs"
- note added: "MOSFETs"
- note added: "Mechanical - Mounting"
- note added: "Motor Control - Driver"
- note added: "Power - Generation"
- note added: "Power - Input"
- note added: "References: Vincent Nguyen: https://github.com/nguyen-v/amulet_controller_kibot SIROJU: https://www.youtube.com/@srj4555"
- note added: "Sensing - Battery"
- note added: "Sensing - Position"
- note added: "Sensing - Temperature"
- note added: "USER - LEDs"
- note removed: "${VARIANT} ${RELEASE_DATE}"
- note removed: "Add a comment here"
- note removed: "Block Diagram"
- note removed: "CHECKED - There shouldn't be any mistakes. Contact the engineer if you find any."
- note removed: "DESIGN CONSIDERATIONS"
- note removed: "DRAFT - Very early stage of schematic, ignore details."
- note removed: "PRELIMINARY - Close to final schematic."
- note removed: "Power - Sequencing"
- note removed: "RELEASED - A board with this schematic has been sent to production."
- note removed: "Random Sheet 1"
- note removed: "Random Sheet 2"
- note removed: "Revision History"

Commit message: Clean up schematic design notes; export schematic and PCB artwork PDFs
- Remove firmware-only notes (boot sequence, calibration procedure,
  firmware SPI/PWM settings) and template/empty text; keep hardware facts
- Tighten wording of all DESIGN/SPEC/ASSEMBLY/REV 1 notes and resize
  boxes so no note text wraps or overflows
- Re-export schematic PDF
- Add PCB artwork PDFs (combined and one per layer: silk, paste, mask,
  L1-L6 copper), board outline on every page

Co-Authored-By: Claude Opus 5.5 <noreply@anthropic.com>
Other:
- note added: "${RELEASE_DATE}"
- note added: "Variant: Prototype"
- note removed: "${CURRENT_DATE}"
- note removed: "Variant: ${VARIANT}"
Changed lines of the file:
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@@
 	(title_block
 		(title "Cover Page")
-		(date "Last Modified Date")
+		(date "${RELEASE_DATE}")
 		(rev "${REVISION}")
 		(company "${COMPANY}")
@@
 		)
 	)
-	(text "Sensing - Battery"
+	(text "Sensing - Temperature"
 		(exclude_from_sim no)
 		(at 45.72 152.4 0)
@@
 		)
 	)
-	(text "Interface - Interconnects"
+	(text "Mechanical - Mounting"
 		(exclude_from_sim no)
 		(at 144.78 99.06 0)
@@
 		)
 	)
-	(text "Power - Generation\n"
+	(text "Power - Generation"
 		(exclude_from_sim no)
 		(at 45.72 106.68 0)
@@
 		)
 	)
-	(text "${CURRENT_DATE}"
+	(text "${RELEASE_DATE}"
 		(exclude_from_sim no)
 		(at 388.62 40.64 0)
@@
 		)
 	)
-	(text "Variant: ${VARIANT}"
+	(text "Variant: Prototype"
 		(exclude_from_sim no)
 		(at 25.4 58.42 0)
@@
 		)
 	)
-	(text "Sensing - Temperature"
+	(text "Interface - CAN FD"
 		(exclude_from_sim no)
 		(at 144.78 83.82 0)
@@
 		)
 	)
-	(text "USER - LEDs"
+	(text "..........................................."
 		(exclude_from_sim no)
 		(at 144.78 114.3 0)
@@
 		)
 	)
-	(text "Mechanical - Mounting"
+	(text "USER - LEDs"
 		(exclude_from_sim no)
 		(at 144.78 106.68 0)
@@
 		)
 	)
-	(text "Interface - CAN FD"
+	(text "Interface - Interconnects"
 		(exclude_from_sim no)
 		(at 144.78 91.44 0)
@@
 		)
 	)
-	(text_box "Metadata can be set in File → Schematic Setup → Project → Text Variables"
-		(exclude_from_sim no)
-		(at 27.94 306.07 0)
-		(size 119.38 6.35)
-		(margins 1.9049 1.9049 1.9049 1.9049)
-		(stroke
-			(width -0.0001)
-			(type default)
-		)
-		(fill
-			(type none)
-		)
-		(effects
-			(font
-				(size 2.54 2.54)
-				(thickness 0.381)
-				(bold yes)
-				(color 0 0 0 1)
-			)
-			(justify right top)
-		)
-	)
