File: Schematics/Interface_Interconnects.kicad_sch (KiCad schematic)
At the start: 32 parts, among them J1 Conn_01x04_MountingPin, J10 Conn_01x02_MountingPin, J11 Conn_01x02_MountingPin, J2 Conn_01x03, J3 Conn_01x04_MountingPin, J4 Conn_01x04_MountingPin, J5 Conn_01x04_MountingPin, J6 Conn_01x07_MountingPin, J7 Conn_01x05, SW1 SW_Push_DPDT

Commit message: Clean up schematic design notes; export schematic and PCB artwork PDFs
- Remove firmware-only notes (boot sequence, calibration procedure,
  firmware SPI/PWM settings) and template/empty text; keep hardware facts
- Tighten wording of all DESIGN/SPEC/ASSEMBLY/REV 1 notes and resize
  boxes so no note text wraps or overflows
- Re-export schematic PDF
- Add PCB artwork PDFs (combined and one per layer: silk, paste, mask,
  L1-L6 copper), board outline on every page

Co-Authored-By: Claude Opus 5.5 <noreply@anthropic.com>
Other:
- company: (none) -> ${COMPANY}
- title: (none) -> Interface - Interconnects
Changed lines of the file:
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@@
 	(generator_version "10.0")
 	(paper "A3")
+	(title_block
+		(title "Interface - Interconnects")
+		(date "${RELEASE_DATE}")
+		(rev "${REVISION}")
+		(company "${COMPANY}")
+	)
 	(rectangle
 		(start 138.43 144.78)
@@
 		)
 	)
-	(text_box "DESIGN NOTE:\nLoop closed = PC3 low = run;\n  \nLoop open OR cable unplugged = PC3 high = hardware break."
-		(exclude_from_sim no)
-		(at 57.15 123.7632 0)
-		(size 34.29 14.6668)
-		(margins 0.9525 0.9525 0.9525 0.9525)
-		(stroke
-			(width 0.508)
-			(type solid)
-			(color 0 0 255 1)
-		)
-		(fill
-			(type color)
-			(color 255 255 255 1)
-		)
-		(effects
-			(font
-				(size 1.27 1.27)
-				(color 0 0 0 1)
-			)
-			(justify left top)
-		)
-	)
-	(text_box "DESIGN NOTE:\nJ6 shares SPI1 (SCK/MISO/MOSI) with the on-board AS5047P (U1).\nIsolation is by chip select only: U1 on PA4, remote on PC4.\nAS5047P tri-states MISO when CSn is high (datasheet t_OZ), so two\nslaves on one bus is valid - but firmware MUST NOT assert both\nchip selects."
+	(text_box "DESIGN NOTE:\nSHARED SPI1\nJ6 (AUX2) shares SCK/MISO/MOSI with\non-board U1 (AS5047P). Selected by CS\nonly: U1 on PA4, remote on PC4.\nAS5047P tri-states MISO when CSn is\nhigh; only one CS active at a time."
 		(exclude_from_sim no)
 		(at 306.07 160.7462 0)
-		(size 46.99 22.35)
+		(size 46.99 17.78)
 		(margins 0.9525 0.9525 0.9525 0.9525)
 		(stroke
@@
 		)
 	)
-	(text_box "DESIGN NOTE:\n\nNo ESD protection for prototype.\nExpected to be in lab environment."
-		(exclude_from_sim no)
-		(at 25.4 38.1 0)
-		(size 44.45 14.1714)
-		(margins 0.9525 0.9525 0.9525 0.9525)
-		(stroke
-			(width 0.508)
-			(type solid)
-			(color 0 0 255 1)
-		)
-		(fill
-			(type color)
-			(color 255 255 255 1)
-		)
-		(effects
-			(font
-				(size 1.27 1.27)
-				(color 0 0 0 1)
-			)
-			(justify left top)
-		)
-	)
 	(text_box "Temperature"
 		(exclude_from_sim no)
@@
 		)
 	)
-	(text_box "DESIGN NOTE:\nUART PIN NAMING\nNet UART1_TX lands on PB7 = USART1_RX.\nNet UART1_RX lands on PB6 = USART1_TX."
+	(text_box "DESIGN NOTE:\nUART NET NAMING\nUART1_TX -> PB7 (USART1_RX)\nUART1_RX -> PB6 (USART1_TX)"
 		(exclude_from_sim no)
 		(at 293.37 60.2632 0)
-		(size 34.29 14.1714)
+		(size 34.29 11.43)
 		(margins 0.9525 0.9525 0.9525 0.9525)
 		(stroke
@@
 	(text_box "[${#}] Interface - Interconnects"
 		(exclude_from_sim no)
-		(at 134.62 11.43 0)
-		(size 273.05 24.4424)
+		(at 12.7 12.7 0)
+		(size 394.97 24.4424)
 		(margins 5.9999 5.9999 5.9999 5.9999)
 		(stroke
@@
 		)
 	)
-)
+	(text_box "DESIGN NOTE:\nESD PROTECTION\nCAN bus: D4/D7 PESD2CANFD24V on CANH/CANL.\nSWD, UART, I2C, AUX2, NTC and E-stop connectors\nunprotected (prototype, lab use)."
+		(exclude_from_sim no)
+		(at 25.4 54.61 0)
+		(size 55.88 12.70)
+		(margins 0.9525 0.9525 0.9525 0.9525)
+		(stroke
+			(width 0.508)
+			(type solid)
+			(color 0 0 255 1)
+		)
+		(fill
+			(type color)
+			(color 255 255 255 1)
+		)
+		(effects
+			(font
+				(size 1.27 1.27)
+				(color 0 0 0 1)
+			)
+			(justify left top)
+		)
+	)
+	(rectangle
+		(start 22.86 85.09)
+		(end 133.35 177.8)
+		(stroke
+			(width 1)
+			(type default)
+			(color 200 200 200 1)
+		)
+		(fill
+			(type none)
+		)
+	)
+	(text_box "E-Stop"
+		(exclude_from_sim no)
+		(at 22.86 168.7697 0)
+		(size 110.49 7.7603)
+		(margins 1.9049 1.9049 1.9049 1.9049)
+		(stroke
+			(width -0.0001)
+			(type solid)
+		)
+		(fill
+			(type none)
+		)
+		(effects
+			(font
+				(face "Times New Roman")
+				(size 2.54 2.54)
+				(thickness 0.508)
+				(bold yes)
+				(color 162 22 34 1)
+			)
+			(justify bottom)
+		)
+	)
+	(text_box "REV 1 NOTE:\nE-STOP NOT FUNCTIONAL AS DRAWN\nJ11-1 connects directly to DRV_ENABLE; R41/C42 feed\nthe same node into PC3 (ESTOP).\n- Unplugged: R16 100k holds DRV_ENABLE low\n  (driver off = fail-safe).\n- J11 looped to GND: shorts the MCU DRV_ENABLE\n  output; driver cannot be enabled.\n- PC3 only mirrors DRV_ENABLE.\nLeave J11 unplugged; bench supply switch is the\nE-stop. Rev 2: separate E-stop input."
+		(exclude_from_sim no)
+		(at 25.4 88.9 0)
+		(size 57.15 25.40)
+		(margins 0.9525 0.9525 0.9525 0.9525)
+		(stroke
+			(width 0.508)
+			(type solid)
+			(color 255 0 0 1)
+		)
+		(fill
+			(type color)
+			(color 255 255 255 1)
+		)
+		(effects
+			(font
+				(size 1.27 1.27)
+				(color 0 0 0 1)
+			)
+			(justify left top)
+		)
+	)
+	(text_box "DESIGN NOTE:\nCALC - SPLIT TERMINATION (SW1 selects)\nDifferential: R45 + R46 = 120.8 R (spec 120 R +/-10%)\nCommon-mode:  fc = 1/(2*pi*(R45||R46)*C68)\n                 = 1/(2*pi*30.2*47n) = 112 kHz\nEnable (SW1 ON) only at the two bus-end nodes.\nJ4/J5 daisy-chain the bus; J2 (DNP) is an alternate.\nNo common-mode choke: sub-metre harness,\nno certification requirement."
+		(exclude_from_sim no)
+		(at 96.52 186.69 0)
+		(size 64.77 21.59)
+		(margins 0.9525 0.9525 0.9525 0.9525)
+		(stroke
+			(width 0.508)
+			(type solid)
+			(color 0 0 255 1)
+		)
+		(fill
+			(type color)
+			(color 255 255 255 1)
+		)
+		(effects
+			(font
+				(size 1.27 1.27)
+				(color 0 0 0 1)
+			)
+			(justify left top)
+		)
+	))
