File: Schematics/MCU_IOs.kicad_sch (KiCad schematic)
At the start: 45 parts, among them U5 STM32G431RBTx, X1 SMD3225-4

Commit message: Clean up schematic design notes; export schematic and PCB artwork PDFs
- Remove firmware-only notes (boot sequence, calibration procedure,
  firmware SPI/PWM settings) and template/empty text; keep hardware facts
- Tighten wording of all DESIGN/SPEC/ASSEMBLY/REV 1 notes and resize
  boxes so no note text wraps or overflows
- Re-export schematic PDF
- Add PCB artwork PDFs (combined and one per layer: silk, paste, mask,
  L1-L6 copper), board outline on every page

Co-Authored-By: Claude Opus 5.5 <noreply@anthropic.com>
Other:
- company: (none) -> ${COMPANY}
- title: (none) -> MCU - IOs
Changed lines of the file:
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@@
 	(generator_version "10.0")
 	(paper "A3")
+	(title_block
+		(title "MCU - IOs")
+		(date "${RELEASE_DATE}")
+		(rev "${REVISION}")
+		(company "${COMPANY}")
+	)
 	(rectangle
 		(start 302.26 186.69)
@@
 	)
 	(rectangle
-		(start 120.65 170.18)
-		(end 156.21 172.72)
-		(stroke
-			(width 0)
-			(type dot)
-			(color 255 0 0 1)
-		)
-		(fill
-			(type none)
-		)
-	)
-	(rectangle
 		(start 24.13 36.83)
 		(end 201.93 223.52)
@@
 		)
 	)
-	(text_box "DESIGN NOTE:\nCALC - CRYSTAL LOAD\nCL = (C28 x C29)/(C28 + C29) + Cstray\n   = (12 x 12)/24 + ~5 = 11 pF\nSelected a crystal specified for CL = 11-12 pF."
-		(exclude_from_sim no)
-		(at 27.94 141.7593 0)
-		(size 38.1 16.2161)
-		(margins 0.9525 0.9525 0.9525 0.9525)
-		(stroke
-			(width 0.508)
-			(type solid)
-			(color 0 0 255 1)
-		)
-		(fill
-			(type color)
-			(color 255 255 255 1)
-		)
-		(effects
-			(font
-				(size 1.27 1.27)
-				(color 0 0 0 1)
-			)
-			(justify left top)
-		)
-	)
 	(text_box "Analog IO"
 		(exclude_from_sim no)
@@
 		)
 	)
-	(text_box "REVIEW"
-		(exclude_from_sim no)
-		(at 387.35 73.66 0)
-		(size 19.05 6.35)
-		(margins 0.9525 0.9525 0.9525 0.9525)
-		(stroke
-			(width 0.508)
-			(type solid)
-			(color 255 0 0 1)
-		)
-		(fill
-			(type color)
-			(color 255 0 0 1)
-		)
-		(effects
-			(font
-				(size 2.54 2.54)
-				(color 0 0 0 1)
-			)
-			(justify left top)
-		)
-	)
 	(text_box "[${#}] MCU - IOs"
 		(exclude_from_sim no)
@@
 		)
 	)
-	(text_box "SPEC:\nADC CHANNEL MAP\n  FILTER_SOA  PB11  ADC1_IN14 / ADC2_IN14   (both)\n  FILTER_SOB  PB12  ADC1_IN11               (ADC1 only)\n  FILTER_SOC  PB14  ADC1_IN5                (ADC1 only)\n  VBAT_SENSE  PB0   ADC1_IN15\n  TEMP_SENSE  PB1   ADC1_IN12\n  MOT_TEMP    PB2   ADC2_IN12\n\n  Simultaneous dual-ADC sampling MUST pair SOA (on ADC2) with SOB or\n  SOC (on ADC1). Phases B and C can NEVER be sampled simultaneously.\n  Derive the third phase from Ia + Ib + Ic = 0."
-		(exclude_from_sim no)
-		(at 309.88 45.72 0)
-		(size 83.82 38.1)
-		(margins 0.9525 0.9525 0.9525 0.9525)
-		(stroke
-			(width 0.508)
-			(type solid)
-			(color 0 194 0 1)
-		)
-		(fill
-			(type color)
-			(color 255 255 255 1)
-		)
-		(effects
-			(font
-				(size 1.27 1.27)
-				(color 0 0 0 1)
-			)
-			(justify left top)
-		)
-	)
-	(text_box "REVIEW"
-		(exclude_from_sim no)
-		(at 167.64 170.18 0)
-		(size 19.05 6.35)
-		(margins 0.9525 0.9525 0.9525 0.9525)
-		(stroke
-			(width 0.508)
-			(type solid)
-			(color 255 0 0 1)
-		)
-		(fill
-			(type color)
-			(color 255 0 0 1)
-		)
-		(effects
-			(font
-				(size 2.54 2.54)
-				(color 0 0 0 1)
-			)
-			(justify left top)
-		)
-	)
 	(text_box "MCU - STM32G431RBT6"
 		(exclude_from_sim no)
@@
 		)
 	)
-	(text_box "FIRMWARE - MANDATORY AT BOOT\n  1. Program nSWBOOT0 = 0 so BOOT0 comes from the option bit,\n     not PB8 (PB8 = FDCAN1_RX).\n  2. Set PWR_CR3.UCPD1_DBDIS = 1 BEFORE enabling TIM1.\n     PA9/PA10 (PWM_PHASEB_H / PWM_PHASEC_H) are UCPD1_DBCC1/2.\n     A high level enables internal 5.1k pull-downs on PB6 (UART TX)\n     and PB4 (PWR_LED).\n  3. DRV_nFAULT -> PA15 = TIM1_BKIN (AF9). Configure as a hardware\n     break input, not EXTI.\n  4. ESTOP -> PC3 = TIM1_BKIN2 (AF6), active HIGH (loop open)."
-		(exclude_from_sim no)
-		(at 160.02 130.356 0)
-		(size 36.83 42.364)
-		(margins 0.9525 0.9525 0.9525 0.9525)
-		(stroke
-			(width 0.508)
-			(type solid)
-			(color 0 0 255 1)
-		)
-		(fill
-			(type color)
-			(color 255 255 255 1)
-		)
-		(effects
-			(font
-				(size 1.27 1.27)
-				(color 0 0 0 1)
-			)
-			(justify left top)
-		)
-	)
 	(text_box "Testpoints\n"
 		(exclude_from_sim no)
@@
 		)
 	)
-	(polyline
-		(pts
-			(xy 160.02 165.1) (xy 156.21 170.18)
-		)
-		(stroke
-			(width 0)
-			(type dot)
-			(color 255 0 0 1)
-		)
-	)
 	(wire
 		(pts
@@
 		)
 	)
-)
+	(text_box "DESIGN NOTE:\nSHARED-FUNCTION PINS\nPB8 = BOOT0 and FDCAN1_RX.\nPA9/PA10 (PWM_PHASEB_H / PWM_PHASEC_H) are\n  UCPD1 dead-battery pins: a high level enables\n  5.1k pull-downs on PB6 (UART TX) and PB4 (PWR_LED).\nDRV_nFAULT -> PA15 (TIM1_BKIN).\nESTOP -> PC3 (TIM1_BKIN2)."
+		(exclude_from_sim no)
+		(at 27.94 171.45 0)
+		(size 63.5 19.05)
+		(margins 0.9525 0.9525 0.9525 0.9525)
+		(stroke
+			(width 0.508)
+			(type solid)
+			(color 0 0 255 1)
+		)
+		(fill
+			(type color)
+			(color 255 255 255 1)
+		)
+		(effects
+			(font
+				(size 1.27 1.27)
+				(color 0 0 0 1)
+			)
+			(justify left top)
+		)
+	)
+	(text_box "DESIGN NOTE:\nCALC - CRYSTAL LOAD\nX1 25 MHz HSE\nCL = C28*C29/(C28+C29)\n     + Cstray\n   = 12x12/24 + ~5 = 11 pF\nCrystal spec CL = 11-12 pF."
+		(exclude_from_sim no)
+		(at 27.94 139.7 0)
+		(size 35.56 17.78)
+		(margins 0.9525 0.9525 0.9525 0.9525)
+		(stroke
+			(width 0.508)
+			(type solid)
+			(color 0 0 255 1)
+		)
+		(fill
+			(type color)
+			(color 255 255 255 1)
+		)
+		(effects
+			(font
+				(size 1.27 1.27)
+				(color 0 0 0 1)
+			)
+			(justify left top)
+		)
+	)
+	(text_box "SPEC:\nADC CHANNEL MAP\n  FILTER_SOA  PB11  ADC1_IN14 / ADC2_IN14   (both)\n  FILTER_SOB  PB12  ADC1_IN11               (ADC1 only)\n  FILTER_SOC  PB14  ADC1_IN5                (ADC1 only)\n  VBAT_SENSE  PB0   ADC1_IN15\n  TEMP_SENSE  PB1   ADC1_IN12\n  MOT_TEMP    PB2   ADC2_IN12\nSOB and SOC are both ADC1-only: phases B and C\ncannot be sampled simultaneously."
+		(exclude_from_sim no)
+		(at 309.88 45.72 0)
+		(size 80.01 22.86)
+		(margins 0.9525 0.9525 0.9525 0.9525)
+		(stroke
+			(width 0.508)
+			(type solid)
+			(color 0 194 0 1)
+		)
+		(fill
+			(type color)
+			(color 255 255 255 1)
+		)
+		(effects
+			(font
+				(size 1.27 1.27)
+				(color 0 0 0 1)
+			)
+			(justify left top)
+		)
+	))
