File: Schematics/Position.kicad_sch (KiCad schematic)
At the start: 2 parts, among them U1 AS5047P-ATSM

Commit message: Clean up schematic design notes; export schematic and PCB artwork PDFs
- Remove firmware-only notes (boot sequence, calibration procedure,
  firmware SPI/PWM settings) and template/empty text; keep hardware facts
- Tighten wording of all DESIGN/SPEC/ASSEMBLY/REV 1 notes and resize
  boxes so no note text wraps or overflows
- Re-export schematic PDF
- Add PCB artwork PDFs (combined and one per layer: silk, paste, mask,
  L1-L6 copper), board outline on every page

Co-Authored-By: Claude Opus 5.5 <noreply@anthropic.com>
Other:
- company: (none) -> ${COMPANY}
- title: (none) -> Sensing - Position
Changed lines of the file:
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@@
 	(generator_version "10.0")
 	(paper "A4")
+	(title_block
+		(title "Sensing - Position")
+		(date "${RELEASE_DATE}")
+		(rev "${REVISION}")
+		(company "${COMPANY}")
+	)
 	(rectangle
 		(start 38.1 38.1)
@@
 			)
 			(justify bottom)
-		)
-	)
-	(text_box "SPEC:  \nU1  AS5047P-ATSM  ams  TSSOP-14\n14-bit (16384 counts/rev) | up to 28 krpm | DAEC\nSPI slave, mode 1 (CPOL=0, CPHA=1), up to 10 MHz, MSB first\n"
-		(exclude_from_sim no)
-		(at 83.82 52.0701 0)
-		(size 63.5 12.6999)
-		(margins 0.9525 0.9525 0.9525 0.9525)
-		(stroke
-			(width 0.508)
-			(type solid)
-			(color 0 194 0 1)
-		)
-		(fill
-			(type color)
-			(color 255 255 255 1)
-		)
-		(effects
-			(font
-				(size 1.27 1.27)
-				(color 0 0 0 1)
-			)
-			(justify left top)
-		)
-	)
-	(text_box "ASSEMBLY:\n  Package centre must be concentric with the rotor axis within\n  [FILL] mm. Diametric magnet, air gap per datasheet magnetic\n  characteristics.\n  No ferrous hardware or switching copper within [FILL] mm."
-		(exclude_from_sim no)
-		(at 153.67 67.3101 0)
-		(size 68.58 16.5099)
-		(margins 0.9525 0.9525 0.9525 0.9525)
-		(stroke
-			(width 0.508)
-			(type solid)
-			(color 255 153 0 1)
-		)
-		(fill
-			(type color)
-			(color 255 255 255 1)
-		)
-		(effects
-			(font
-				(size 1.27 1.27)
-				(color 0 0 0 1)
-			)
-			(justify left top)
-		)
-	)
-	(text_box "DESIGN NOTE:\nVDD and VDD3V tied for 3.3 V operation\nTEST (pin 5) tied to GND - required\nA/B/I/U/V/W left open - permitted (datasheet pin note 5)"
-		(exclude_from_sim no)
-		(at 83.82 71.1201 0)
-		(size 63.5 12.6999)
-		(margins 0.9525 0.9525 0.9525 0.9525)
-		(stroke
-			(width 0.508)
-			(type solid)
-			(color 0 0 255 1)
-		)
-		(fill
-			(type color)
-			(color 255 255 255 1)
-		)
-		(effects
-			(font
-				(size 1.27 1.27)
-				(color 0 0 0 1)
-			)
-			(justify left top)
-		)
-	)
-	(text_box "REVIEW"
-		(exclude_from_sim no)
-		(at 179.07 82.55 0)
-		(size 19.05 6.35)
-		(margins 0.9525 0.9525 0.9525 0.9525)
-		(stroke
-			(width 0.508)
-			(type solid)
-			(color 255 0 0 1)
-		)
-		(fill
-			(type color)
-			(color 255 0 0 1)
-		)
-		(effects
-			(font
-				(size 2.54 2.54)
-				(color 0 0 0 1)
-			)
-			(justify left top)
 		)
 	)
@@
 		)
 	)
-)
+	(text_box "ASSEMBLY:\nMAGNET PLACEMENT (datasheet reference values)\nDiametric magnet, ref. N35H 8 mm dia x 3 mm.\nAir gap ~2.0 mm, Bz 35-70 mT.\nCentre on U1 package within 0.5 mm\n(INL +/-1.2 deg at 500 um offset).\nKeep ferrous hardware and phase/bus copper away."
+		(exclude_from_sim no)
+		(at 158.75 52.07 0)
+		(size 54.61 17.78)
+		(margins 0.9525 0.9525 0.9525 0.9525)
+		(stroke
+			(width 0.508)
+			(type solid)
+			(color 255 153 0 1)
+		)
+		(fill
+			(type color)
+			(color 255 255 255 1)
+		)
+		(effects
+			(font
+				(size 1.27 1.27)
+				(color 0 0 0 1)
+			)
+			(justify left top)
+		)
+	)
+	(text_box "SPEC:\nU1  AS5047P-ATSM  ams  TSSOP-14\n14-bit (16384 counts/rev) | up to 28 krpm | DAEC\nSPI slave, mode 1 (CPOL=0, CPHA=1), up to 10 MHz, MSB first"
+		(exclude_from_sim no)
+		(at 83.82 52.0701 0)
+		(size 69.85 11.43)
+		(margins 0.9525 0.9525 0.9525 0.9525)
+		(stroke
+			(width 0.508)
+			(type solid)
+			(color 0 194 0 1)
+		)
+		(fill
+			(type color)
+			(color 255 255 255 1)
+		)
+		(effects
+			(font
+				(size 1.27 1.27)
+				(color 0 0 0 1)
+			)
+			(justify left top)
+		)
+	)
+	(text_box "DESIGN NOTE:\nVDD and VDD3V tied for 3.3 V operation\nTEST (pin 5) tied to GND - required\nA/B/I/U/V/W left open - permitted (datasheet pin note 5)"
+		(exclude_from_sim no)
+		(at 83.82 71.1201 0)
+		(size 66.04 11.43)
+		(margins 0.9525 0.9525 0.9525 0.9525)
+		(stroke
+			(width 0.508)
+			(type solid)
+			(color 0 0 255 1)
+		)
+		(fill
+			(type color)
+			(color 255 255 255 1)
+		)
+		(effects
+			(font
+				(size 1.27 1.27)
+				(color 0 0 0 1)
+			)
+			(justify left top)
+		)
+	))
