File: Schematics/Power_Input.kicad_sch (KiCad schematic)
At the start: 3 parts

Commit message: Clean up schematic design notes; export schematic and PCB artwork PDFs
- Remove firmware-only notes (boot sequence, calibration procedure,
  firmware SPI/PWM settings) and template/empty text; keep hardware facts
- Tighten wording of all DESIGN/SPEC/ASSEMBLY/REV 1 notes and resize
  boxes so no note text wraps or overflows
- Re-export schematic PDF
- Add PCB artwork PDFs (combined and one per layer: silk, paste, mask,
  L1-L6 copper), board outline on every page

Co-Authored-By: Claude Opus 5.5 <noreply@anthropic.com>
Other:
- company: (none) -> ${COMPANY}
- title: (none) -> Power - Input
Changed lines of the file:
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@@
 	(generator_version "10.0")
 	(paper "A4")
+	(title_block
+		(title "Power - Input")
+		(date "${RELEASE_DATE}")
+		(rev "${REVISION}")
+		(company "${COMPANY}")
+	)
 	(rectangle
 		(start 73.66 53.34)
@@
 		)
 	)
-	(text_box "ACCEPTED RISK:\nD1 clamps at 82.4 V. Downstream absolute maximums:\nDRV8323 VM/VDRAIN   65 V\nLMR36520 VIN        65 V\nTLV75733 VIN       5.5 V (fed from +5V, not exposed)\nD1 therefore does NOT protect the board against an event large\nenough to engage it.\n\nSOLUTION:\nUpstream PDB handles protection"
+	(text_box "ACCEPTED RISK:\nD1 clamps at 82.4 V, above\ndownstream abs max:\n  DRV8323 VM/VDRAIN  65 V\n  LMR36520 VIN       65 V\nD1 cannot protect the board\nfrom an event large enough\nto engage it.\nMitigation: overvoltage\nprotection in upstream PDB."
 		(exclude_from_sim no)
 		(at 85.09 67.31 0)
-		(size 35.56 29.21)
+		(size 35.56 22.86)
 		(margins 0.9525 0.9525 0.9525 0.9525)
 		(stroke
@@
 		)
 	)
-	(text_box "ASSEMBLY:\nD3.2mm solder pad, no connector"
+	(text_box "ASSEMBLY:\n3.2 mm dia\nsolder pad,\nno connector"
 		(exclude_from_sim no)
 		(at 125.73 67.31 0)
-		(size 16.51 10.16)
+		(size 16.51 11.43)
 		(margins 0.9525 0.9525 0.9525 0.9525)
 		(stroke
