File: Schematics/Sensing_Temperature.kicad_sch (KiCad schematic)
At the start: 9 parts

Commit message: Clean up schematic design notes; export schematic and PCB artwork PDFs
- Remove firmware-only notes (boot sequence, calibration procedure,
  firmware SPI/PWM settings) and template/empty text; keep hardware facts
- Tighten wording of all DESIGN/SPEC/ASSEMBLY/REV 1 notes and resize
  boxes so no note text wraps or overflows
- Re-export schematic PDF
- Add PCB artwork PDFs (combined and one per layer: silk, paste, mask,
  L1-L6 copper), board outline on every page

Co-Authored-By: Claude Opus 5.5 <noreply@anthropic.com>
Other:
- company: (none) -> ${COMPANY}
- title: (none) -> Sensing - Temperature
Changed lines of the file:
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@@
 	(generator_version "10.0")
 	(paper "A4")
+	(title_block
+		(title "Sensing - Temperature")
+		(date "${RELEASE_DATE}")
+		(rev "${REVISION}")
+		(company "${COMPANY}")
+	)
 	(text_box "[${#}] Sensing - Temperature"
 		(exclude_from_sim no)
@@
 				(color 162 22 34 1)
 			)
-		)
-	)
-	(text_box "On-Board 10k NTC"
-		(exclude_from_sim no)
-		(at 68.58 126.8597 0)
-		(size 58.42 7.7603)
-		(margins 1.9049 1.9049 1.9049 1.9049)
-		(stroke
-			(width -0.0001)
-			(type solid)
-		)
-		(fill
-			(type none)
-		)
-		(effects
-			(font
-				(face "Times New Roman")
-				(size 2.54 2.54)
-				(thickness 0.508)
-				(bold yes)
-				(color 162 22 34 1)
-			)
-			(justify bottom)
-		)
-	)
-	(text_box "DESIGN NOTE:\nCALC - 10K NTC ON-BOARD NCP18XH103J03RB\n  V = 3.3 x R38/(NTC + R38)\n    -10 C (~42k)  -> 0.63 V\n     25 C (10k)   -> 1.65 V\n    100 C (~680R) -> 3.09 V\n  Self-heat: I = 165 uA, P = 0.27 mW, <0.1 C rise. Negligible."
-		(exclude_from_sim no)
-		(at 30.48 92.71 0)
-		(size 43.18 21.59)
-		(margins 0.9525 0.9525 0.9525 0.9525)
-		(stroke
-			(width 0.508)
-			(type solid)
-			(color 0 0 255 1)
-		)
-		(fill
-			(type color)
-			(color 255 255 255 1)
-		)
-		(effects
-			(font
-				(size 1.27 1.27)
-				(color 0 0 0 1)
-			)
-			(justify left top)
-		)
-	)
-	(text_box "Motor NTC\n"
-		(exclude_from_sim no)
-		(at 140.97 126.8597 0)
-		(size 58.42 7.7603)
-		(margins 1.9049 1.9049 1.9049 1.9049)
-		(stroke
-			(width -0.0001)
-			(type solid)
-		)
-		(fill
-			(type none)
-		)
-		(effects
-			(font
-				(face "Times New Roman")
-				(size 2.54 2.54)
-				(thickness 0.508)
-				(bold yes)
-				(color 162 22 34 1)
-			)
-			(justify bottom)
-		)
-	)
-	(text_box "DESIGN NOTE:\nCALC - MOTOR (external NTC on top, R39 2k to GND)\n  V = 3.3 x 2k/(NTC + 2k)\n     25 C (10k)   -> 0.55 V\n    100 C (~680R) -> 2.46 V"
-		(exclude_from_sim no)
-		(at 200.66 87.63 0)
-		(size 43.18 16.51)
-		(margins 0.9525 0.9525 0.9525 0.9525)
-		(stroke
-			(width 0.508)
-			(type solid)
-			(color 0 0 255 1)
-		)
-		(fill
-			(type color)
-			(color 255 255 255 1)
-		)
-		(effects
-			(font
-				(size 1.27 1.27)
-				(color 0 0 0 1)
-			)
-			(justify left top)
 		)
 	)
@@
 		)
 	)
-)
+	(rectangle
+		(start 25.4 54.61)
+		(end 132.08 139.7)
+		(stroke
+			(width 1)
+			(type default)
+			(color 200 200 200 1)
+		)
+		(fill
+			(type none)
+		)
+	)
+	(text_box "On-Board 10k NTC"
+		(exclude_from_sim no)
+		(at 25.4 130.6697 0)
+		(size 106.68 7.7603)
+		(margins 1.9049 1.9049 1.9049 1.9049)
+		(stroke
+			(width -0.0001)
+			(type solid)
+		)
+		(fill
+			(type none)
+		)
+		(effects
+			(font
+				(face "Times New Roman")
+				(size 2.54 2.54)
+				(thickness 0.508)
+				(bold yes)
+				(color 162 22 34 1)
+			)
+			(justify bottom)
+		)
+	)
+	(rectangle
+		(start 135.89 54.61)
+		(end 271.78 139.7)
+		(stroke
+			(width 1)
+			(type default)
+			(color 200 200 200 1)
+		)
+		(fill
+			(type none)
+		)
+	)
+	(text_box "Motor NTC (via J10)"
+		(exclude_from_sim no)
+		(at 135.89 130.6697 0)
+		(size 135.89 7.7603)
+		(margins 1.9049 1.9049 1.9049 1.9049)
+		(stroke
+			(width -0.0001)
+			(type solid)
+		)
+		(fill
+			(type none)
+		)
+		(effects
+			(font
+				(face "Times New Roman")
+				(size 2.54 2.54)
+				(thickness 0.508)
+				(bold yes)
+				(color 162 22 34 1)
+			)
+			(justify bottom)
+		)
+	)
+	(text_box "DESIGN NOTE:\nCALC - MOTOR NTC (external NTC on top,\nR39 2k to GND)\n  V = 3.3 x 2k/(NTC + 2k)\n     25 C (10k)   -> 0.55 V\n    100 C (~680R) -> 2.46 V\nDZ3 clamps the off-board line to 3.3 V."
+		(exclude_from_sim no)
+		(at 200.66 87.63 0)
+		(size 46.99 17.78)
+		(margins 0.9525 0.9525 0.9525 0.9525)
+		(stroke
+			(width 0.508)
+			(type solid)
+			(color 0 0 255 1)
+		)
+		(fill
+			(type color)
+			(color 255 255 255 1)
+		)
+		(effects
+			(font
+				(size 1.27 1.27)
+				(color 0 0 0 1)
+			)
+			(justify left top)
+		)
+	)
+	(text_box "DESIGN NOTE:\nCALC - 10K NTC ON-BOARD (R37)\nNCP18XH103J03RB, R38 10k to GND\n  V = 3.3 x R38/(NTC + R38)\n    -10 C (~42k)  -> 0.63 V\n     25 C (10k)   -> 1.65 V\n    100 C (~680R) -> 3.09 V\nSelf-heat: I = 165 uA, P = 0.27 mW,\n  <0.1 C rise. Negligible."
+		(exclude_from_sim no)
+		(at 27.94 88.9 0)
+		(size 43.18 21.59)
+		(margins 0.9525 0.9525 0.9525 0.9525)
+		(stroke
+			(width 0.508)
+			(type solid)
+			(color 0 0 255 1)
+		)
+		(fill
+			(type color)
+			(color 255 255 255 1)
+		)
+		(effects
+			(font
+				(size 1.27 1.27)
+				(color 0 0 0 1)
+			)
+			(justify left top)
+		)
+	))
