File: Schematics/USER_LEDs.kicad_sch (KiCad schematic)
At the start: 6 parts

Commit message: Clean up schematic design notes; export schematic and PCB artwork PDFs
- Remove firmware-only notes (boot sequence, calibration procedure,
  firmware SPI/PWM settings) and template/empty text; keep hardware facts
- Tighten wording of all DESIGN/SPEC/ASSEMBLY/REV 1 notes and resize
  boxes so no note text wraps or overflows
- Re-export schematic PDF
- Add PCB artwork PDFs (combined and one per layer: silk, paste, mask,
  L1-L6 copper), board outline on every page

Co-Authored-By: Claude Opus 5.5 <noreply@anthropic.com>
Other:
- company: (none) -> ${COMPANY}
- title: (none) -> USER - LEDs
Changed lines of the file:
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@@
 	(generator_version "10.0")
 	(paper "A4")
+	(title_block
+		(title "USER - LEDs")
+		(date "${RELEASE_DATE}")
+		(rev "${REVISION}")
+		(company "${COMPANY}")
+	)
 	(text_box "[${#}] User - LEDs"
 		(exclude_from_sim no)
@@
 		)
 	)
-)
+	(rectangle
+		(start 76.2 58.42)
+		(end 215.9 137.16)
+		(stroke
+			(width 1)
+			(type default)
+			(color 200 200 200 1)
+		)
+		(fill
+			(type none)
+		)
+	)
+	(text_box "Status LEDs"
+		(exclude_from_sim no)
+		(at 76.2 128.1297 0)
+		(size 139.7 7.7603)
+		(margins 1.9049 1.9049 1.9049 1.9049)
+		(stroke
+			(width -0.0001)
+			(type solid)
+		)
+		(fill
+			(type none)
+		)
+		(effects
+			(font
+				(face "Times New Roman")
+				(size 2.54 2.54)
+				(thickness 0.508)
+				(bold yes)
+				(color 162 22 34 1)
+			)
+			(justify bottom)
+		)
+	))
